Commit message: add collision and inertia to model
use xacro later

File: robot_model.urdf (robot description, URDF)
Before this commit: robot crackvac, 9 links, 8 joints
Links:
- link base_link: mass None -> 7.0; geometry collision box size=0.4 0.4 0.2; visual box size=0.4 0.4 0.2
- link bl_wheel: mass None -> 0.079; geometry collision cylinder length=0.03 radius=0.04; visual cylinder length=0.03 radius=0.04
- link br_wheel: mass None -> 0.079; geometry collision cylinder length=0.03 radius=0.04; visual cylinder length=0.03 radius=0.04
- link fl_wheel: mass None -> 0.079; geometry collision cylinder length=0.03 radius=0.04; visual cylinder length=0.03 radius=0.04
- link fr_wheel: mass None -> 0.079; geometry collision cylinder length=0.03 radius=0.04; visual cylinder length=0.03 radius=0.04
