Commit message: urdf calculate inertia with properties

File: sim/urdf/robot_model.urdf.xacro (robot description, xacro)
@@ -16,15 +16,24 @@
     <xacro:property name="wheel_base" value="0.4064"/>
     <xacro:property name="wheel_base_half" value="${wheel_base / 2}"/>
-    <xacro:property name="robot_mass" value="7.0"/> <!-- mass unit: kg-->
+    <xacro:property name="chassis_depth" value="0.2032"/>
+    <xacro:property name="chassis_mass" value="7.0"/> <!-- mass unit: kg-->
+    <xacro:property name="wheel_mass" value="0.186"/> <!-- mass unit: kg-->
     <!-- macros -->
     <link name="dummy_link">
         <collision>
             <geometry>
-                <box size="0.4 0.4 0.2"/>
+                <box size="${wheel_base} ${wheel_base} ${chassis_depth}"/>
             </geometry>
         </collision>
         <inertial>
-            <mass value="${robot_mass}"/>
-            <inertia ixx="0.187" ixy="0.0" ixz="0.0" iyy="0.117" iyz="0.0" izz="0.117"/>
+            <mass value="${chassis_mass}"/>
+            <inertia
+                ixx="${1/12 * chassis_mass * (wheel_base * wheel_base + chassis_depth * chassis_depth)}"
+                ixy="0.0"
+                ixz="0.0"
+                iyy="${1/12 * chassis_mass * (wheel_base * wheel_base + chassis_depth * chassis_depth)}"
+                iyz="0.0"
+                izz="${1/12 * chassis_mass * (wheel_base * wheel_base + wheel_base * wheel_base)}"
+            />
         </inertial>
     </link>
@@ -37,7 +46,7 @@
             <visual>
                 <geometry>
-                    <box size="0.4 0.4 0.2"/>
+                    <box size="${wheel_base} ${wheel_base} ${chassis_depth}"/>
                 </geometry>
-                <origin xyz="0.0 0.0 0.1" rpy="0.0 0.0 0.0"/>
+                <origin xyz="0.0 0.0 ${chassis_depth / 2}" rpy="0.0 0.0 0.0"/>
                 <material name="grey"/>
             </visual>
@@ -64,5 +73,5 @@
             <collision>
                 <geometry>
-                    <cylinder radius="0.04" length="0.03"/>
+                    <cylinder radius="${wheel_radius}" length="${wheel_width}"/>
                 </geometry>
                 <origin xyz="0 0 0" rpy="1.57 0 0"/>
@@ -70,5 +79,12 @@
             <inertial>
                 <mass value="0.079"/>
-                <inertia ixx="0.002291" ixy="0.0" ixz="0.0" iyy="0.002291" iyz="0.0" izz="0.0000632"/>
+                <inertia
+                    ixx="${1/12 * wheel_mass* (3 * wheel_radius * wheel_radius + wheel_width * wheel_width)}"
+                    ixy="0.0"
+                    ixz="0.0"
+                    iyy="${1/12 * wheel_mass* (3 * wheel_radius * wheel_radius + wheel_width * wheel_width)}"
+                    iyz="0.0"
+                    izz="${1/2 * wheel_mass * wheel_radius * wheel_radius}"
+                />
             </inertial>
         </link>

Commit message: launch gazebo with controller, remove wheel collision

File: sim/urdf/robot_model.urdf.xacro (robot description, xacro)
@@ -12,11 +12,11 @@
     </material>
     <!-- constants -->
-    <xacro:property name="wheel_radius" value="0.04"/> <!-- length unit: m-->
+    <xacro:property name="wheel_radius" value="0.04"/> <!-- length unit m-->
     <xacro:property name="wheel_width" value="0.03"/>
     <xacro:property name="wheel_base" value="0.4064"/>
     <xacro:property name="wheel_base_half" value="${wheel_base / 2}"/>
     <xacro:property name="chassis_depth" value="0.2032"/>
-    <xacro:property name="chassis_mass" value="7.0"/> <!-- mass unit: kg-->
-    <xacro:property name="wheel_mass" value="0.186"/> <!-- mass unit: kg-->
+    <xacro:property name="chassis_mass" value="7.0"/> <!-- mass unit kg-->
+    <xacro:property name="wheel_mass" value="0.186"/>
     <!-- macros -->
     <link name="dummy_link">
@@ -75,10 +75,4 @@
                 <material name="black"/>
             </visual>
-            <collision>
-                <geometry>
-                    <cylinder radius="${wheel_radius}" length="${wheel_width}"/>
-                </geometry>
-                <origin xyz="0 0 0" rpy="1.57 0 0"/>
-            </collision>
             <inertial>
                 <mass value="0.079"/>
